File: brd/exampcb-led.sch (KiCad schematic (older format))
At the start: 11 parts, among them P1 POWER, U1 LM358

Commit message: new: dev: nuevo form-factor, cambio divisor y conector USB !wip
Parts:
- removed D1: GREEN, symbol LED
- removed P1: POWER, symbol CONN_01X02
- added J1: XM7D-0512, asrdi-conn:UE25-BEx5-10x, symbol USB_OTG
- added J2: 5V, Connect:1pin, symbol CONN_01X01
- added J3: GND, Connect:1pin, symbol CONN_01X01
- added R6: 82R, Discret:R4-LARGE_PADS, symbol R
- C1: renamed from C2; footprint (none) -> Capacitors_ThroughHole:C_Rect_L7_W2.5_P5; symbol C -> C-RESCUE-exampcb-led
- C2: renamed from C1; footprint (none) -> Capacitors_ThroughHole:C_Rect_L7_W2.5_P5; symbol C -> C-RESCUE-exampcb-led
- D1: renamed from D2; value YELLOW -> LED; footprint (none) -> LEDs:LED-5MM; symbol LED -> LED-RESCUE-exampcb-led
- R1, R3: footprint (none) -> Discret:R4-LARGE_PADS
- R2: value 10k -> 680R; footprint (none) -> Discret:R4-LARGE_PADS
- R4: value 10M -> 10k; footprint (none) -> Discret:R4-LARGE_PADS
- R5: value 82R -> 10M; footprint (none) -> Discret:R4-LARGE_PADS
- U1: footprint (none) -> Housings_DIP:DIP-8__300_ELL
Other:
- moved on the sheet: C2
Changed lines of the file:
@@
 EESchema Schematic File Version 2
+LIBS:exampcb-led-rescue
 LIBS:power
 LIBS:device
@@
 LIBS:memory
 LIBS:xilinx
-LIBS:special
 LIBS:microcontrollers
 LIBS:dsp
@@
 	4450 4150 4650 4150
 Wire Wire Line
-	4450 4050 4450 4250
+	4450 3950 4450 4300
 Wire Wire Line
 	4650 4850 4750 4850
@@
 	4650 3400 4650 4850
 Wire Wire Line
-	4650 3400 4700 3400
+	4650 3400 4800 3400
 Connection ~ 5300 3400
 Wire Wire Line
@@
 	5300 4050 5350 4050
 Wire Wire Line
-	6000 3400 6400 3400
-Wire Wire Line
-	5200 3400 5500 3400
+	5900 3400 6400 3400
+Wire Wire Line
+	5100 3400 5600 3400
 Wire Wire Line
 	5750 4550 5750 4650
 Wire Wire Line
-	8300 4150 8350 4150
-Wire Wire Line
-	3700 4200 3750 4200
-Connection ~ 3750 3900
-Wire Wire Line
-	3750 3800 3750 4100
-Wire Wire Line
-	3750 4400 4000 4400
-Wire Wire Line
-	4000 4400 4000 4350
-Wire Wire Line
-	4000 3950 4000 3900
-Wire Wire Line
-	4000 3900 3750 3900
-Wire Wire Line
-	3750 4200 3750 4500
-Connection ~ 3750 4400
-Wire Wire Line
-	3750 4100 3700 4100
+	8200 4150 8350 4150
+Wire Wire Line
+	3700 4350 4150 4350
+Wire Wire Line
+	4150 3800 4150 4075
+Wire Wire Line
+	7325 3750 7325 3600
+Wire Wire Line
+	7325 3200 7325 3050
+Wire Wire Line
+	4150 4225 4150 4500
+Wire Wire Line
+	4150 3950 3700 3950
 Wire Wire Line
 	8800 4300 8800 4150
@@
 	8800 4150 8750 4150
 Wire Wire Line
-	7700 4150 7800 4150
+	7700 4150 7900 4150
 Wire Wire Line
 	5750 3750 5750 3700
@@
 	6350 4150 6400 4150
 Wire Wire Line
-	5150 4850 5500 4850
-Wire Wire Line
-	6400 4850 6000 4850
+	5150 4850 5600 4850
+Wire Wire Line
+	6400 4850 5900 4850
 Wire Wire Line
 	6400 3400 6400 4850
@@
 Connection ~ 5300 4850
 Wire Wire Line
-	4450 4800 4450 4650
-Wire Wire Line
-	4450 3550 4450 3450
+	4450 4800 4450 4600
+Wire Wire Line
+	4450 3650 4450 3450
 Wire Wire Line
 	6700 4050 6600 4050
@@
 	6600 4050 6600 5000
 Wire Wire Line
-	5300 5000 6600 5000
-Wire Wire Line
-	5300 4250 5300 5000
+	6600 5000 5300 5000
+Wire Wire Line
+	5300 5000 5300 4250
 Wire Wire Line
 	7100 4550 7100 4650
 $Comp
-L GND #PWR01
+L GND-RESCUE-exampcb-led #PWR01
 U 1 1 4E6F6D7D
 P 7100 4650
@@
 $EndComp
 $Comp
-L GND #PWR04
+L GND-RESCUE-exampcb-led #PWR04
 U 1 1 4E6F6B62
 P 4450 4800
@@
 $EndComp
 $Comp
-L GND #PWR05
+L GND-RESCUE-exampcb-led #PWR05
 U 1 1 4E6F6A5E
 P 5750 4650
@@
 $EndComp
 $Comp
-L GND #PWR07
+L GND-RESCUE-exampcb-led #PWR07
 U 1 1 4E6F69D4
 P 8800 4300
@@
 $EndComp
 $Comp
-L GND #PWR08
+L GND-RESCUE-exampcb-led #PWR08
 U 1 1 4E6F68CB
-P 3750 4500
-F 0 "#PWR08" H 3750 4500 30  0001 C CNN
-F 1 "GND" H 3750 4430 30  0001 C CNN
-F 2 "" H 3750 4500 60  0001 C CNN
-F 3 "" H 3750 4500 60  0001 C CNN
-	1    3750 4500
+P 4150 4500
+F 0 "#PWR08" H 4150 4500 30  0001 C CNN
+F 1 "GND" H 4150 4430 30  0001 C CNN
+F 2 "" H 4150 4500 60  0001 C CNN
+F 3 "" H 4150 4500 60  0001 C CNN
+	1    4150 4500
 	1    0    0    -1
 $EndComp
@@
 L VCC #PWR09
 U 1 1 4E6F68C1
-P 3750 3800
-F 0 "#PWR09" H 3750 3900 30  0001 C CNN
-F 1 "VCC" H 3750 3900 30  0000 C CNN
-F 2 "" H 3750 3800 60  0001 C CNN
-F 3 "" H 3750 3800 60  0001 C CNN
-	1    3750 3800
+P 4150 3800
+F 0 "#PWR09" H 4150 3900 30  0001 C CNN
+F 1 "VCC" H 4150 3900 30  0000 C CNN
+F 2 "" H 4150 3800 60  0001 C CNN
+F 3 "" H 4150 3800 60  0001 C CNN
+	1    4150 3800
 	1    0    0    -1
 $EndComp
@@
 F 0 "U1" H 7150 4350 60  0000 L CNN
 F 1 "LM358" H 7150 3900 60  0000 L CNN
-F 2 "" H 7200 4150 60  0001 C CNN
+F 2 "Housings_DIP:DIP-8__300_ELL" H 7200 4150 60  0001 C CNN
 F 3 "" H 7200 4150 60  0001 C CNN
 	2    7200 4150
@@
 $EndComp
 $Comp
-L LED D2
+L LED-RESCUE-exampcb-led D1
 U 1 1 4E6F6841
 P 8550 4150
-F 0 "D2" H 8550 4250 50  0000 C CNN
-F 1 "YELLOW" H 8550 4050 50  0000 C CNN
-F 2 "" H 8550 4150 60  0001 C CNN
+F 0 "D1" H 8550 4250 50  0000 C CNN
+F 1 "LED" H 8550 4050 50  0000 C CNN
+F 2 "LEDs:LED-5MM" H 8550 4150 60  0001 C CNN
 F 3 "" H 8550 4150 60  0001 C CNN
 	1    8550 4150
@@
 $EndComp
 $Comp
-L LED D1
-U 1 1 4E6F683D
-P 4450 4450
-F 0 "D1" V 4550 4250 50  0000 C CNN
-F 1 "GREEN" V 4650 4300 50  0000 C CNN
-F 2 "" H 4450 4450 60  0001 C CNN
-F 3 "" H 4450 4450 60  0001 C CNN
-	1    4450 4450
-	0    1    1    0
-$EndComp
-$Comp
-L C C1
+L C-RESCUE-exampcb-led C2
 U 1 1 4E6F6828
-P 4000 4150
-F 0 "C1" H 4050 4250 50  0000 L CNN
-F 1 "10nF" H 4050 4050 50  0000 L CNN
-F 2 "" H 4000 4150 60  0001 C CNN
-F 3 "" H 4000 4150 60  0001 C CNN
-	1    4000 4150
-	1    0    0    -1
-$EndComp
-$Comp
-L C C2
+P 7325 3400
+F 0 "C2" H 7375 3500 50  0000 L CNN
+F 1 "10nF" H 7375 3300 50  0000 L CNN
+F 2 "Capacitors_ThroughHole:C_Rect_L7_W2.5_P5" H 7325 3400 60  0001 C CNN
+F 3 "" H 7325 3400 60  0001 C CNN
+	1    7325 3400
+	1    0    0    -1
+$EndComp
+$Comp
+L C-RESCUE-exampcb-led C1
 U 1 1 4E6F6825
 P 4950 4850
-F 0 "C2" V 4850 4950 50  0000 L CNN
-F 1 "100nF" V 5000 5050 50  0000 L CNN
-F 2 "" H 4950 4850 60  0001 C CNN
+F 0 "C1" V 4850 4950 50  0000 L CNN
+F 1 "100nF" V 5000 4925 50  0000 L CNN
+F 2 "Capacitors_ThroughHole:C_Rect_L7_W2.5_P5" H 4950 4850 60  0001 C CNN
 F 3 "" H 4950 4850 60  0001 C CNN
 	1    4950 4850
-	0    1    1    0
-$EndComp
-$Comp
-L R R5
-U 1 1 4E6F681C
-P 8050 4150
-F 0 "R5" V 8130 4150 50  0000 C CNN
-F 1 "82R" V 8050 4150 50  0000 C CNN
-F 2 "" H 8050 4150 60  0001 C CNN
-F 3 "" H 8050 4150 60  0001 C CNN
-	1    8050 4150
-	0    1    1    0
-$EndComp
-$Comp
-L R R1
-U 1 1 4E6F681A
-P 4450 3800
-F 0 "R1" H 4250 3950 50  0000 C CNN
-F 1 "680R" H 4300 3850 50  0000 C CNN
-F 2 "" H 4450 3800 60  0001 C CNN
-F 3 "" H 4450 3800 60  0001 C CNN
-	1    4450 3800
-	1    0    0    -1
-$EndComp
-$Comp
-L R R3
-U 1 1 4E6F6816
-P 5750 3400
-F 0 "R3" V 5830 3400 50  0000 C CNN
-F 1 "10k" V 5750 3400 50  0000 C CNN
-F 2 "" H 5750 3400 60  0001 C CNN
-F 3 "" H 5750 3400 60  0001 C CNN
-	1    5750 3400
-	0    1    1    0
-$EndComp
-$Comp
-L R R4
-U 1 1 4E6F6814
-P 5750 4850
-F 0 "R4" V 5830 4850 50  0000 C CNN
-F 1 "10M" V 5750 4850 50  0000 C CNN
-F 2 "" H 5750 4850 60  0001 C CNN
-F 3 "" H 5750 4850 60  0001 C CNN
-	1    5750 4850
-	0    1    1    0
-$EndComp
-$Comp
-L R R2
-U 1 1 4E6F680F
-P 4950 3400
-F 0 "R2" V 5030 3400 50  0000 C CNN
-F 1 "10k" V 4950 3400 50  0000 C CNN
-F 2 "" H 4950 3400 60  0001 C CNN
-F 3 "" H 4950 3400 60  0001 C CNN
-	1    4950 3400
 	0    1    1    0
 $EndComp
@@
 F 0 "U1" H 5800 4350 60  0000 L CNN
 F 1 "LM358" H 5800 3900 60  0000 L CNN
-F 2 "" H 5850 4150 60  0001 C CNN
+F 2 "Housings_DIP:DIP-8__300_ELL" H 5850 4150 60  0001 C CNN
 F 3 "" H 5850 4150 60  0001 C CNN
 	1    5850 4150
@@
 $EndComp
 $Comp
-L CONN_01X02 P1
-U 1 1 54823C27
-P 3500 4150
-F 0 "P1" H 3500 4300 50  0000 C CNN
-F 1 "POWER" V 3600 4150 50  0000 C CNN
-F 2 "" H 3500 4150 60  0000 C CNN
-F 3 "" H 3500 4150 60  0000 C CNN
-	1    3500 4150
+L R R2
+U 1 1 55C68113
+P 4450 4450
+F 0 "R2" V 4530 4450 50  0000 C CNN
+F 1 "680R" V 4450 4450 50  0000 C CNN
+F 2 "Discret:R4-LARGE_PADS" V 4380 4450 30  0001 C CNN
+F 3 "" H 4450 4450 30  0000 C CNN
+	1    4450 4450
+	1    0    0    -1
+$EndComp
+$Comp
+L R R1
+U 1 1 55C6821C
+P 4450 3800
+F 0 "R1" V 4530 3800 50  0000 C CNN
+F 1 "680R" V 4450 3800 50  0000 C CNN
+F 2 "Discret:R4-LARGE_PADS" V 4380 3800 30  0001 C CNN
+F 3 "" H 4450 3800 30  0000 C CNN
+	1    4450 3800
+	1    0    0    -1
+$EndComp
+$Comp
+L R R3
+U 1 1 55C68253
+P 4950 3400
+F 0 "R3" V 5030 3400 50  0000 C CNN
+F 1 "10k" V 4950 3400 50  0000 C CNN
+F 2 "Discret:R4-LARGE_PADS" V 4880 3400 30  0001 C CNN
+F 3 "" H 4950 3400 30  0000 C CNN
+	1    4950 3400
+	0    1    1    0
+$EndComp
+$Comp
+L R R4
+U 1 1 55C68292
+P 5750 3400
+F 0 "R4" V 5830 3400 50  0000 C CNN
+F 1 "10k" V 5750 3400 50  0000 C CNN
+F 2 "Discret:R4-LARGE_PADS" V 5680 3400 30  0001 C CNN
+F 3 "" H 5750 3400 30  0000 C CNN
+	1    5750 3400
+	0    1    1    0
+$EndComp
+$Comp
+L R R5
+U 1 1 55C682D5
+P 5750 4850
+F 0 "R5" V 5830 4850 50  0000 C CNN
+F 1 "10M" V 5750 4850 50  0000 C CNN
+F 2 "Discret:R4-LARGE_PADS" V 5680 4850 30  0001 C CNN
+F 3 "" H 5750 4850 30  0000 C CNN
+	1    5750 4850
+	0    1    1    0
+$EndComp
+$Comp
+L R R6
+U 1 1 55C68334
+P 8050 4150
+F 0 "R6" V 8130 4150 50  0000 C CNN
+F 1 "82R" V 8050 4150 50  0000 C CNN
+F 2 "Discret:R4-LARGE_PADS" V 7980 4150 30  0001 C CNN
+F 3 "" H 8050 4150 30  0000 C CNN
+	1    8050 4150
+	0    1    1    0
+$EndComp
+$Comp
+L USB_OTG J1
+U 1 1 55C71503
+P 3400 4150
+F 0 "J1" V 3725 4025 50  0000 C CNN
+F 1 "XM7D-0512" H 3400 4350 50  0000 C CNN
+F 2 "asrdi-conn:UE25-BEx5-10x" V 3350 4050 60  0001 C CNN
+F 3 "" V 3350 4050 60  0000 C CNN
+	1    3400 4150
+	0    -1   1    0
+$EndComp
+$Comp
+L GND-RESCUE-exampcb-led #PWR010
+U 1 1 55C71703
+P 7325 3750
+F 0 "#PWR010" H 7325 3750 30  0001 C CNN
+F 1 "GND" H 7325 3680 30  0001 C CNN
+F 2 "" H 7325 3750 60  0001 C CNN
+F 3 "" H 7325 3750 60  0001 C CNN
+	1    7325 3750
+	1    0    0    -1
+$EndComp
+$Comp
+L VCC #PWR011
+U 1 1 55C71732
+P 7325 3050
+F 0 "#PWR011" H 7325 3150 30  0001 C CNN
+F 1 "VCC" H 7325 3150 30  0000 C CNN
+F 2 "" H 7325 3050 60  0001 C CNN
+F 3 "" H 7325 3050 60  0001 C CNN
+	1    7325 3050
+	1    0    0    -1
+$EndComp
+Wire Wire Line
+	4150 4075 4100 4075
+Connection ~ 4150 3950
+Wire Wire Line
+	4100 4225 4150 4225
+Connection ~ 4150 4350
+$Comp
+L CONN_01X01 J2
+U 1 1 564235C2
+P 3900 4075
+F 0 "J2" H 3900 4175 50  0000 C CNN
+F 1 "5V" V 4000 4075 50  0000 C CNN
+F 2 "Connect:1pin" H 3900 4075 60  0001 C CNN
+F 3 "" H 3900 4075 60  0000 C CNN
+	1    3900 4075
 	-1   0    0    1
 $EndComp
+$Comp
+L CONN_01X01 J3
+U 1 1 564236DF
+P 3900 4225
+F 0 "J3" H 3900 4325 50  0000 C CNN
+F 1 "GND" V 4000 4225 50  0000 C CNN
+F 2 "Connect:1pin" H 3900 4225 60  0001 C CNN
+F 3 "" H 3900 4225 60  0000 C CNN
+	1    3900 4225
+	-1   0    0    1
+$EndComp
